File: Demo Project 01.sch (KiCad schematic (older format))
At the start: 81 parts, among them J2 Conn_02x03_Odd_Even, J3 Conn_02x13_Odd_Even, J4 Conn_02x05_Odd_Even, J5 Screw_Terminal_01x01, J6 Screw_Terminal_01x01, J8 Conn_01x02, U1 L7805

Commit message: - Cleaned up schematic layout by creating dedicated sheet for codec as   well as analog input filters in addition to the main Teensy sheet - Added schematics for all AIN filters based on codec datasheet - Added dedicated 3v3 supply and gave all supplies power flags. Created   dedicated digital/analog GND as well as recommended 3v3A for codec power
Parts:
- removed C? (x4): 100N, symbol Device:C
- removed C? (x16): C, symbol Device:C
- removed C? (x7): 0.1uf, symbol Device:C_Small
- removed C? (x4): 0.01uf, symbol Device:C_Small
- removed C? (x2): 10uf, symbol Device:CP1
- removed C?: 100uf, symbol Device:CP1
- removed C?: 22uf, symbol Device:CP1
- removed C? (x5): 4.7uf, symbol Device:CP1
- removed J2: Conn_02x03_Odd_Even, Connector_PinHeader_2.54mm:PinHeader_2x03_P2.54mm_Vertical, symbol Connector_Generic:Conn_02x03_Odd_Even
- removed R? (x2): 10R PF RAD, symbol Device:R
- removed R? (x16): R, symbol Device:R
- removed U? (x12): TL072, symbol Amplifier_Operational:TL072
- removed U?: CS42448-CQZ, QFP50P1200X1200X160-64N, symbol imoptooo:CS42448-CQZ
- added C? (x2): 10u, symbol Device:C
- added R?: 10k, symbol Device:R
- added R? (x2): R, symbol Device:R
- added U?: LP3853ES-3.3_NOPB, TS5B, symbol LP3853ES-3.3NOPB:LP3853ES-3.3_NOPB
Connections:
- net labels added: +3.3V, +5V, CODEC_INT, CODEC_~RST, ETH_LED, ETH_R+, ETH_R-, ETH_T+, ETH_T-, GNDD, GNDPWR, USBDEV_D+, USBDEV_D-, USBHOST_D+, USBHOST_D-
- net labels removed: AIN1+, AIN1-, AIN2+, AIN2-, AIN3+, AIN3-, AIN4+, AIN4-, AOUT1+, AOUT1-, AOUT2+, AOUT2-, AOUT3+, AOUT3-, AOUT4+, AOUT4-, AOUT5+, AOUT5-, AOUT6+, AOUT6-, CODEC_MCLK, RESET, SPI_CLK, SPI_MISO, SPI_MOSI, VCC
- wire segments 124 -> 90
- no-connect marks 8 -> 4
Other:
- moved on the sheet: C6, C7, J3, J4, J5, J6, J8, U1, U?
